Commit message: Set the mass of VI-Sensor to zero, for simple simulation in Gazebo (without the dynamic model of vi-sensor)

File: rotors_description/urdf/component_snippets.xacro (robot description, xacro)
@@ -491,5 +491,6 @@
       </visual>
       <inertial>
-        <mass value="0.13" />
+        <!-- <mass value="0.13" /> -->
+        <mass value="1e-5" />
         <origin xyz="0 0 0" rpy="0 0 0" />
         <inertia ixx="1e-6" ixy="0" ixz="0" iyy="1e-6" iyz="0" izz="1e-6" />

File: rotors_description/urdf/vi_sensor_base.xacro (robot description, xacro)
@@ -18,7 +18,9 @@
     </visual>
     <inertial>
-      <mass value="100" />
+      <!-- <mass value="100" /> -->
+      <mass value="0" />
       <origin xyz="0 0 0" rpy="0 0 0" />
-      <inertia ixx="1" ixy="0" ixz="0" iyy="1" iyz="0" izz="1" />
+      <!-- <inertia ixx="1" ixy="0" ixz="0" iyy="1" iyz="0" izz="1" /> -->
+      <inertia ixx="0" ixy="0" ixz="0" iyy="0" iyz="0" izz="0" />
     </inertial>
   </link>
