Commit message: Minor changes for compatible in MoveIt

File: rotors_description/urdf/firefly.xacro (robot description, xacro)
@@ -18,5 +18,5 @@
 <robot name="firefly" xmlns:xacro="http://ros.org/wiki/xacro">
   <!-- Properties -->
-  <xacro:property name="namespace" value="$(arg mav_name)" />
+  <xacro:property name="namespace" value="firefly" />
   <xacro:property name="rotor_velocity_slowdown_sim" value="10" />
   <xacro:property name="use_mesh_file" value="true" />

File: rotors_description/urdf/firefly_base.xacro (robot description, xacro)
@@ -24,8 +24,10 @@
   <!-- Mount an ADIS16448 IMU. -->
   <xacro:default_imu namespace="${namespace}" parent_link="${namespace}/base_link" />
-  <xacro:if value="$(arg enable_ground_truth)">
+  <!-- <xacro:if value="$(arg enable_ground_truth)"> -->
+  <xacro:if value="true">
     <xacro:ground_truth_imu_and_odometry namespace="${namespace}" parent_link="${namespace}/base_link" />
   </xacro:if>
-  <xacro:if value="$(arg enable_logging)">
+  <!-- <xacro:if value="$(arg enable_logging)"> -->
+  <xacro:if value="false">
     <!-- Instantiate a logger -->
     <xacro:bag_plugin_macro

File: rotors_description/urdf/hummingbird.xacro (robot description, xacro)
@@ -19,5 +19,5 @@
   <!-- Properties (Taken from Novel Dynamic Inversion Architecture Design
 for Quadrocopter Control by Jian Wang et al.) -->
-  <xacro:property name="namespace" value="$(arg mav_name)" />
+  <xacro:property name="namespace" value="hummingbird" />
   <xacro:property name="rotor_velocity_slowdown_sim" value="10" />
   <xacro:property name="use_mesh_file" value="true" />
